File: Electronica/EAGLE ADAPTADOR/AdaptadorAcceso.sch (EAGLE design)
At the start: 9 parts

Commit message: PCB terminado - A revisar
Connections:
- net N$4 renamed GND_FUENTE
- removed net GND_OPTO: OK1B.EMIT, OK2A.EMIT, OK2B.EMIT, SV2.3
- net GNDA: now also OK1B.EMIT, OK2A.EMIT, OK2B.EMIT, SV2.3
Changed lines of the file:
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@@
 <part name="+3V3" library="supply1" deviceset="+3V3" device=""/>
 <part name="GND2" library="supply1" deviceset="GNDA" device=""/>
+<part name="GND3" library="supply1" deviceset="GNDA" device=""/>
+<part name="GND4" library="supply1" deviceset="GNDA" device=""/>
+<part name="GND7" library="supply1" deviceset="GNDA" device=""/>
+<part name="GND8" library="supply1" deviceset="GNDA" device=""/>
 </parts>
 <sheets>
@@
 <attribute name="VALUE" x="143.34" y="0.5" size="1.778" layer="96" rot="R180"/>
 </instance>
+<instance part="GND3" gate="1" x="20.32" y="-33.02" smashed="yes" rot="R270">
+<attribute name="VALUE" x="18.28" y="-36.66" size="1.778" layer="96" rot="R90"/>
+</instance>
+<instance part="GND4" gate="1" x="27.94" y="20.32" smashed="yes">
+<attribute name="VALUE" x="31.58" y="18.28" size="1.778" layer="96" rot="R180"/>
+</instance>
+<instance part="GND7" gate="1" x="27.94" y="35.56" smashed="yes">
+<attribute name="VALUE" x="31.58" y="33.52" size="1.778" layer="96" rot="R180"/>
+</instance>
+<instance part="GND8" gate="1" x="27.94" y="53.34" smashed="yes">
+<attribute name="VALUE" x="31.58" y="51.3" size="1.778" layer="96" rot="R180"/>
+</instance>
 </instances>
 <busses>
@@
 <pinref part="GND2" gate="1" pin="GNDA"/>
 </segment>
+<segment>
+<pinref part="SV2" gate="1" pin="3"/>
+<pinref part="GND3" gate="1" pin="GNDA"/>
+<wire x1="38.1" y1="-33.02" x2="22.86" y2="-33.02" width="0.1524" layer="91"/>
+</segment>
+<segment>
+<pinref part="OK2" gate="B" pin="EMIT"/>
+<wire x1="12.7" y1="22.86" x2="27.94" y2="22.86" width="0.1524" layer="91"/>
+<pinref part="GND4" gate="1" pin="GNDA"/>
+</segment>
+<segment>
+<pinref part="OK2" gate="A" pin="EMIT"/>
+<wire x1="12.7" y1="38.1" x2="27.94" y2="38.1" width="0.1524" layer="91"/>
+<pinref part="GND7" gate="1" pin="GNDA"/>
+</segment>
+<segment>
+<pinref part="OK1" gate="B" pin="EMIT"/>
+<wire x1="12.7" y1="55.88" x2="27.94" y2="55.88" width="0.1524" layer="91"/>
+<pinref part="GND8" gate="1" pin="GNDA"/>
+</segment>
 </net>
 <net name="+3V3" class="1">
@@
 </segment>
 </net>
-<net name="IO16" class="0">
+<net name="IO16" class="2">
 <segment>
 <pinref part="J1" gate="G$1" pin="8"/>
@@
 </segment>
 </net>
-<net name="IO18" class="0">
+<net name="IO18" class="2">
 <segment>
 <pinref part="J4" gate="A" pin="3"/>
@@
 </segment>
 </net>
-<net name="IO40" class="0">
+<net name="IO40" class="2">
 <segment>
 <pinref part="J1" gate="G$1" pin="11"/>
@@
 </segment>
 </net>
-<net name="DATA_RTC" class="0">
+<net name="DATA_RTC" class="2">
 <segment>
 <pinref part="RTC" gate="G$1" pin="2"/>
@@
 </segment>
 </net>
-<net name="CLOCK_RTC" class="0">
+<net name="CLOCK_RTC" class="2">
 <segment>
 <pinref part="RTC" gate="G$1" pin="3"/>
@@
 </segment>
 </net>
-<net name="N$4" class="0">
+<net name="GND_FUENTE" class="0">
 <segment>
 <pinref part="CON_FUENTE" gate="1" pin="1"/>
@@
 <wire x1="-5.08" y1="38.1" x2="-27.94" y2="38.1" width="0.1524" layer="91"/>
 <junction x="-27.94" y="38.1"/>
-</segment>
-</net>
-<net name="C_OPTO2" class="0">
+<label x="-45.72" y="68.58" size="1.778" layer="95"/>
+</segment>
+</net>
+<net name="C_OPTO2" class="2">
 <segment>
 <pinref part="OK2" gate="A" pin="COL"/>
@@
 </segment>
 </net>
-<net name="C_OPTO1" class="0">
+<net name="C_OPTO1" class="2">
 <segment>
 <pinref part="OK1" gate="B" pin="COL"/>
@@
 </segment>
 </net>
-<net name="C_OPTO3" class="0">
+<net name="C_OPTO3" class="2">
 <segment>
 <pinref part="OK2" gate="B" pin="COL"/>
@@
 </segment>
 </net>
-<net name="GND_OPTO" class="0">
-<segment>
-<pinref part="OK2" gate="B" pin="EMIT"/>
-<wire x1="12.7" y1="22.86" x2="27.94" y2="22.86" width="0.1524" layer="91"/>
-<label x="27.94" y="22.86" size="1.27" layer="95" xref="yes"/>
-</segment>
-<segment>
-<pinref part="OK2" gate="A" pin="EMIT"/>
-<wire x1="12.7" y1="38.1" x2="27.94" y2="38.1" width="0.1524" layer="91"/>
-<label x="27.94" y="38.1" size="1.27" layer="95" xref="yes"/>
-</segment>
-<segment>
-<pinref part="OK1" gate="B" pin="EMIT"/>
-<wire x1="12.7" y1="55.88" x2="27.94" y2="55.88" width="0.1524" layer="91"/>
-<label x="27.94" y="55.88" size="1.27" layer="95" xref="yes"/>
-</segment>
-<segment>
-<pinref part="SV2" gate="1" pin="3"/>
-<wire x1="38.1" y1="-33.02" x2="25.4" y2="-33.02" width="0.1524" layer="91"/>
-<label x="25.4" y="-33.02" size="1.27" layer="95" rot="R180" xref="yes"/>
-</segment>
-</net>
-<net name="IO17" class="0">
+<net name="IO17" class="2">
 <segment>
 <pinref part="J4" gate="A" pin="2"/>
@@
 </segment>
 </net>
-<net name="IO39" class="0">
+<net name="IO39" class="2">
 <segment>
 <pinref part="J1" gate="G$1" pin="12"/>
@@
 </segment>
 </net>
-<net name="IO33" class="0">
+<net name="IO33" class="2">
 <segment>
 <pinref part="J1" gate="G$1" pin="6"/>
@@
 </segment>
 </net>
-<net name="IO48" class="0">
+<net name="IO48" class="2">
 <segment>
 <pinref part="MOD.EFAISA" gate="G$1" pin="7"/>
@@
 </segment>
 </net>
-<net name="IO47" class="0">
+<net name="IO47" class="2">
 <segment>
 <pinref part="MOD.EFAISA" gate="G$1" pin="6"/>
@@
 </segment>
 </net>
-<net name="IO46" class="0">
+<net name="IO46" class="2">
 <segment>
 <pinref part="MOD.EFAISA" gate="G$1" pin="5"/>
@@
 </segment>
 </net>
-<net name="IO45" class="0">
+<net name="IO45" class="2">
 <segment>
 <pinref part="MOD.EFAISA" gate="G$1" pin="4"/>
@@
 </segment>
 </net>
-<net name="IO21" class="0">
+<net name="IO21" class="2">
 <segment>
 <pinref part="MOD.EFAISA" gate="G$1" pin="3"/>
@@
 </segment>
 </net>
-<net name="IO42" class="0">
+<net name="IO42" class="2">
 <segment>
 <pinref part="MOD.EFAISA" gate="G$1" pin="2"/>
@@
 </segment>
 </net>
-<net name="IO41" class="0">
+<net name="IO41" class="2">
 <segment>
 <pinref part="MOD.EFAISA" gate="G$1" pin="1"/>

Commit message: Actualizacion PCB - A revisar
Parts:
- renumbered CON_FUENTE to COM_FUENTE
Changed lines of the file:
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@@
 <part name="OK2" library="optocoupler" library_urn="urn:adsk.eagle:library:320" deviceset="ILD610" device="" package3d_urn="urn:adsk.eagle:package:21941/1"/>
 <part name="RTC" library="con-lstb" library_urn="urn:adsk.eagle:library:162" deviceset="MA05-1" device="" package3d_urn="urn:adsk.eagle:package:8332/1"/>
-<part name="CON_FUENTE" library="con-lstb" library_urn="urn:adsk.eagle:library:162" deviceset="MA04-1" device="" package3d_urn="urn:adsk.eagle:package:8337/1"/>
+<part name="COM_FUENTE" library="con-lstb" library_urn="urn:adsk.eagle:library:162" deviceset="MA04-1" device="" package3d_urn="urn:adsk.eagle:package:8337/1"/>
 <part name="+3V3" library="supply1" deviceset="+3V3" device=""/>
 <part name="GND2" library="supply1" deviceset="GNDA" device=""/>
@@
 <attribute name="NAME" x="97.79" y="8.382" size="1.778" layer="95"/>
 </instance>
-<instance part="CON_FUENTE" gate="1" x="-53.34" y="73.66" smashed="yes">
+<instance part="COM_FUENTE" gate="1" x="-53.34" y="73.66" smashed="yes">
 <attribute name="VALUE" x="-54.61" y="63.5" size="1.778" layer="96"/>
 <attribute name="NAME" x="-54.61" y="79.502" size="1.778" layer="95"/>
@@
 <net name="N$1" class="0">
 <segment>
-<pinref part="CON_FUENTE" gate="1" pin="4"/>
+<pinref part="COM_FUENTE" gate="1" pin="4"/>
 <wire x1="-45.72" y1="76.2" x2="-12.7" y2="76.2" width="0.1524" layer="91"/>
 <wire x1="-12.7" y1="76.2" x2="-12.7" y2="60.96" width="0.1524" layer="91"/>
@@
 <net name="N$2" class="0">
 <segment>
-<pinref part="CON_FUENTE" gate="1" pin="3"/>
+<pinref part="COM_FUENTE" gate="1" pin="3"/>
 <wire x1="-45.72" y1="73.66" x2="-15.24" y2="73.66" width="0.1524" layer="91"/>
 <pinref part="OK2" gate="A" pin="A"/>
@@
 <net name="N$3" class="0">
 <segment>
-<pinref part="CON_FUENTE" gate="1" pin="2"/>
+<pinref part="COM_FUENTE" gate="1" pin="2"/>
 <wire x1="-45.72" y1="71.12" x2="-20.32" y2="71.12" width="0.1524" layer="91"/>
 <wire x1="-20.32" y1="71.12" x2="-20.32" y2="27.94" width="0.1524" layer="91"/>
@@
 <net name="GND_FUENTE" class="0">
 <segment>
-<pinref part="CON_FUENTE" gate="1" pin="1"/>
+<pinref part="COM_FUENTE" gate="1" pin="1"/>
 <wire x1="-45.72" y1="68.58" x2="-27.94" y2="68.58" width="0.1524" layer="91"/>
 <wire x1="-27.94" y1="68.58" x2="-27.94" y2="55.88" width="0.1524" layer="91"/>
