File: Electronica/EAGLE ADAPTADOR/AdaptadorAcceso.sch (EAGLE design)
At the start: 9 parts

Commit message: PCB terminado, archivos Gerber generados
Changed lines of the file:
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@@
 <wire x1="-7.62" y1="-38.1" x2="0" y2="-38.1" width="0.1524" layer="91"/>
 <wire x1="0" y1="-38.1" x2="0" y2="-35.56" width="0.1524" layer="91"/>
+<wire x1="0" y1="-38.1" x2="10.16" y2="-38.1" width="0.1524" layer="91"/>
+<junction x="0" y="-38.1"/>
 </segment>
 <segment>
