File: Electronica/EAGLE ADAPTADOR/AdaptadorAcceso.brd (EAGLE design)
At the start: 160.5 x 111 mm, 9 parts

Commit message: Inicio de routeo
Parts:
- removed SV4: (no value), con-lstb:MA04-1
- added CON_FUENTE: (no value), con-lstb:MA04-1
- moved RTC 59.2 mm to (21.0, 42.2), turned to 180 degrees
- moved OK1 31.2 mm to (55.2, 45.0), turned to 180 degrees
- moved OK2 7.04 mm to (43.2, 44.8), turned to 180 degrees
Connections:
- net N$1: now also CON_FUENTE.4; no longer SV4.4
- net N$2: now also CON_FUENTE.3; no longer SV4.3
- net N$3: now also CON_FUENTE.2; no longer SV4.2
- net N$4: now also CON_FUENTE.1; no longer SV4.1
Routing:
- net N$4: track 0.00 -> 36.6 mm
- net DATA_RTC: track 0.00 -> 19.1 mm
- net N$3: track 0.00 -> 18.7 mm
- net N$2: track 0.00 -> 17.7 mm
- net N$1: track 0.00 -> 14.6 mm

Commit message: PCB terminado - A revisar
Parts:
- moved CON_FUENTE 61.0 mm to (88.0, 11.8), turned to 270 degrees
- moved OK1 38.4 mm to (71.0, 10.0), turned to 90 degrees
- moved OK2 35.7 mm to (70.8, 22.0), turned to 90 degrees
- moved SV1 2.30 mm to (27.0, 35.2)
- moved SV2 2.30 mm to (27.2, 17.2)
- moved RTC 0.56 mm to (20.5, 42.0), turned to 0 degrees
- moved J4 0.25 mm to (56.4, 17.6)
Connections:
- net N$4 renamed GND_FUENTE
- removed net GND_OPTO: OK1.6, OK2.6, OK2.8, SV2.3
- net GNDA: now also OK1.6, OK2.6, OK2.8, SV2.3
Routing:
- net IO21: track 0.00 -> 85.5 mm
- net IO17: track 0.00 -> 60.3 mm
- net IO18: track 0.00 -> 58.2 mm
- net IO39: track 0.00 -> 48.8 mm, vias 0 -> 1
- net C_OPTO3: track 0.00 -> 41.2 mm
- net IO48: track 0.00 -> 39.9 mm
- net C_OPTO2: track 0.00 -> 38.6 mm
- net IO41: track 0.00 -> 36.9 mm
- net IO46: track 0.00 -> 36.9 mm
- net IO42: track 0.00 -> 36.8 mm
- net IO45: track 0.00 -> 36.6 mm
- net IO47: track 0.00 -> 36.5 mm
- net IO16: track 0.00 -> 32.9 mm
- net +3V3: track 0.00 -> 29.7 mm
- net IO40: track 0.00 -> 29.1 mm
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- added copper zone on layer 16, net GNDA
Other:
- board size 160.5 x 111 mm -> 95.8 x 50.5 mm

Commit message: Actualizacion PCB - A revisar
Parts:
- removed CON_FUENTE: (no value), con-lstb:MA04-1
- added COM_FUENTE: (no value), con-lstb:MA04-1
- moved OK2 53.6 mm to (19.5, 37.8), turned to 270 degrees
- moved OK1 46.2 mm to (34.2, 38.0), turned to 270 degrees
- moved RTC 24.8 mm to (45.0, 38.0), turned to 90 degrees
- moved J1 13.3 mm to (29.4, 23.1)
- moved J4 13.3 mm to (43.1, 17.9)
- moved MOD.EFAISA 13.3 mm to (29.4, 7.10)
- moved SV1 9.38 mm to (34.0, 29.0)
- moved SV2 9.38 mm to (34.2, 11.0)
Connections:
- net GND_FUENTE: now also COM_FUENTE.1; no longer CON_FUENTE.1
- net N$1: now also COM_FUENTE.4; no longer CON_FUENTE.4
- net N$2: now also COM_FUENTE.3; no longer CON_FUENTE.3
- net N$3: now also COM_FUENTE.2; no longer CON_FUENTE.2
Routing:
- net IO41: track 36.9 -> 93.6 mm
- net IO42: track 36.8 -> 83.9 mm
- net IO45: track 36.6 -> 70.2 mm
- net C_OPTO2: track 38.6 -> 70.6 mm
- net IO39: track 48.8 -> 18.3 mm, vias 1 -> 0
- net IO18: track 58.2 -> 31.9 mm
- net IO16: track 32.9 -> 7.13 mm
- net IO17: track 60.3 -> 34.7 mm, vias 0 -> 1
- net IO33: track 13.4 -> 38.7 mm
- net IO46: track 36.9 -> 61.3 mm
- net C_OPTO3: track 41.2 -> 17.3 mm
- net C_OPTO1: track 22.3 -> 44.3 mm
- net N$1: track 14.6 -> 30.6 mm
- net IO21: track 85.5 -> 69.6 mm, vias 0 -> 1
- net DATA_RTC: track 25.0 -> 9.12 mm
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Other:
- board size 95.8 x 50.5 mm -> 60 x 49 mm
- board text added: "EFAISA Cont. de Acceso Ind. Argentina"
- board text removed: "EFAISAS Cont. de Acceso Ind. Argentina"

Commit message: PCB terminado - A revisar
Parts:
- moved RTC 1.00 mm to (45.0, 39.0)
Routing:
- net DATA_RTC: track 9.12 -> 10.3 mm
Changed lines of the file:
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@@
 <attribute name="VALUE" x="18.865" y="41.306" size="1.27" layer="27" ratio="10" rot="R270"/>
 </element>
-<element name="RTC" library="con-lstb" library_urn="urn:adsk.eagle:library:162" package="MA05-1" package3d_urn="urn:adsk.eagle:package:8332/1" value="" x="45" y="38" smashed="yes" rot="R90">
-<attribute name="MF" value="" x="45" y="38" size="1.778" layer="27" rot="R90" display="off"/>
-<attribute name="MPN" value="" x="45" y="38" size="1.778" layer="27" rot="R90" display="off"/>
-<attribute name="NAME" x="43.349" y="31.65" size="1.27" layer="25" ratio="10" rot="R90"/>
-<attribute name="OC_FARNELL" value="unknown" x="45" y="38" size="1.778" layer="27" rot="R90" display="off"/>
-<attribute name="OC_NEWARK" value="unknown" x="45" y="38" size="1.778" layer="27" rot="R90" display="off"/>
-<attribute name="POPULARITY" value="29" x="45" y="38" size="1.778" layer="27" rot="R90" display="off"/>
-<attribute name="VALUE" x="47.921" y="35.46" size="1.27" layer="27" ratio="10" rot="R90"/>
+<element name="RTC" library="con-lstb" library_urn="urn:adsk.eagle:library:162" package="MA05-1" package3d_urn="urn:adsk.eagle:package:8332/1" value="" x="45" y="39" smashed="yes" rot="R90">
+<attribute name="MF" value="" x="45" y="39" size="1.778" layer="27" rot="R90" display="off"/>
+<attribute name="MPN" value="" x="45" y="39" size="1.778" layer="27" rot="R90" display="off"/>
+<attribute name="NAME" x="43.349" y="32.65" size="1.27" layer="25" ratio="10" rot="R90"/>
+<attribute name="OC_FARNELL" value="unknown" x="45" y="39" size="1.778" layer="27" rot="R90" display="off"/>
+<attribute name="OC_NEWARK" value="unknown" x="45" y="39" size="1.778" layer="27" rot="R90" display="off"/>
+<attribute name="POPULARITY" value="29" x="45" y="39" size="1.778" layer="27" rot="R90" display="off"/>
+<attribute name="VALUE" x="47.921" y="36.46" size="1.27" layer="27" ratio="10" rot="R90"/>
 </element>
 <element name="COM_FUENTE" library="con-lstb" library_urn="urn:adsk.eagle:library:162" package="MA04-1" package3d_urn="urn:adsk.eagle:package:8337/1" value="" x="5.75" y="37.75" smashed="yes" rot="R90">
@@
 <wire x1="20.03" y1="29.90558125" x2="21.85721875" y2="31.7328" width="0.8" layer="16"/>
 <wire x1="20.03" y1="29.90558125" x2="20.03" y2="29" width="0.8" layer="16"/>
-<wire x1="45" y1="32.92" x2="43.8128" y2="31.7328" width="0.9" layer="16"/>
-<wire x1="43.8128" y1="31.7328" x2="21.85721875" y2="31.7328" width="0.9" layer="16"/>
+<wire x1="45" y1="33.92" x2="42.8128" y2="31.7328" width="0.9" layer="16"/>
+<wire x1="42.8128" y1="31.7328" x2="21.85721875" y2="31.7328" width="0.9" layer="16"/>
 </signal>
 <signal name="IO16" class="2">
@@
 <contactref element="RTC" pad="2"/>
 <contactref element="SV1" pad="15"/>
-<wire x1="47.5828" y1="34.07065" x2="46.19345" y2="35.46" width="0.5" layer="16"/>
-<wire x1="45" y1="35.46" x2="46.19345" y2="35.46" width="0.5" layer="16"/>
-<wire x1="47.5828" y1="34.07065" x2="47.5828" y2="32.26935" width="0.5" layer="16"/>
+<wire x1="47.5828" y1="35.32065" x2="46.44345" y2="36.46" width="0.5" layer="16"/>
+<wire x1="45" y1="36.46" x2="46.44345" y2="36.46" width="0.5" layer="16"/>
+<wire x1="47.5828" y1="35.32065" x2="47.5828" y2="32.26935" width="0.5" layer="16"/>
 <wire x1="45.43" y1="30.11655" x2="45.43" y2="29" width="0.5" layer="16"/>
 <wire x1="47.5828" y1="32.26935" x2="45.43" y2="30.11655" width="0.5" layer="16"/>
@@
 <contactref element="SV1" pad="16"/>
 <wire x1="47.589" y1="37.853" x2="47.603" y2="37.853" width="0.5" layer="16"/>
-<wire x1="47.603" y1="37.853" x2="47.456" y2="38" width="0.5" layer="16"/>
-<wire x1="45" y1="38" x2="47.456" y2="38" width="0.5" layer="16"/>
+<wire x1="47.603" y1="37.853" x2="46.456" y2="39" width="0.5" layer="16"/>
+<wire x1="45" y1="39" x2="46.456" y2="39" width="0.5" layer="16"/>
 <wire x1="47.589" y1="37.853" x2="49.25" y2="36.192" width="0.5" layer="16"/>
 <wire x1="47.97" y1="30.72" x2="47.97" y2="29" width="0.5" layer="16"/>
