File: Hardware/EAGLE ADAPTADOR/AdaptadorAcceso.sch (EAGLE design)
At the start: 9 parts

Commit message: Access Adaptation Board Correction
Connections:
- net IO18: now also J4.1; no longer J4.3
Changed lines of the file:
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@@
 <net name="IO18" class="2">
 <segment>
-<pinref part="J4" gate="A" pin="3"/>
-<wire x1="-15.24" y1="-68.58" x2="-15.24" y2="-81.28" width="0.1524" layer="91"/>
-<label x="-15.24" y="-81.28" size="1.27" layer="95" rot="R270" xref="yes"/>
+<label x="-20.32" y="-81.28" size="1.27" layer="95" rot="R270" xref="yes"/>
+<pinref part="J4" gate="A" pin="1"/>
+<wire x1="-20.32" y1="-68.58" x2="-20.32" y2="-81.28" width="0.1524" layer="91"/>
 </segment>
 <segment>

Commit message: Adaptation Board Modifcation, Modifed pins in main
Parts:
- OK1, OK2: value ILD610 -> ILD205; device optocoupler:ILD610 -> optocoupler:ILD205
Connections:
- net C_OPTO2: now also SV2.16; no longer SV2.14
- net C_OPTO3: now also SV2.17; no longer SV1.12
Changed lines of the file:
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@@
 <part name="GND1" library="supply1" deviceset="GNDA" device=""/>
 <part name="+3V2" library="supply1" deviceset="+3V3" device=""/>
-<part name="OK1" library="optocoupler" library_urn="urn:adsk.eagle:library:320" deviceset="ILD610" device="" package3d_urn="urn:adsk.eagle:package:21941/1"/>
-<part name="OK2" library="optocoupler" library_urn="urn:adsk.eagle:library:320" deviceset="ILD610" device="" package3d_urn="urn:adsk.eagle:package:21941/1"/>
 <part name="RTC" library="con-lstb" library_urn="urn:adsk.eagle:library:162" deviceset="MA05-1" device="" package3d_urn="urn:adsk.eagle:package:8332/1"/>
 <part name="COM_FUENTE" library="con-lstb" library_urn="urn:adsk.eagle:library:162" deviceset="MA04-1" device="" package3d_urn="urn:adsk.eagle:package:8337/1"/>
@@
 <part name="GND7" library="supply1" deviceset="GNDA" device=""/>
 <part name="GND8" library="supply1" deviceset="GNDA" device=""/>
+<part name="OK1" library="optocoupler" library_urn="urn:adsk.eagle:library:320" deviceset="ILD2*" device="" package3d_urn="urn:adsk.eagle:package:21945/1" technology="05"/>
+<part name="OK2" library="optocoupler" library_urn="urn:adsk.eagle:library:320" deviceset="ILD2*" device="" package3d_urn="urn:adsk.eagle:package:21945/1" technology="05"/>
 </parts>
 <sheets>
@@
 <attribute name="VALUE" x="71.14" y="-33.06" size="1.778" layer="96" rot="R180"/>
 </instance>
+<instance part="RTC" gate="G$1" x="99.06" y="0" smashed="yes">
+<attribute name="VALUE" x="97.79" y="-10.16" size="1.778" layer="96"/>
+<attribute name="NAME" x="97.79" y="8.382" size="1.778" layer="95"/>
+</instance>
+<instance part="COM_FUENTE" gate="1" x="-53.34" y="73.66" smashed="yes">
+<attribute name="VALUE" x="-54.61" y="63.5" size="1.778" layer="96"/>
+<attribute name="NAME" x="-54.61" y="79.502" size="1.778" layer="95"/>
+</instance>
+<instance part="+3V3" gate="G$1" x="129.54" y="-2.54" smashed="yes">
+<attribute name="VALUE" x="132.1" y="-0.04" size="1.778" layer="96" rot="R180"/>
+</instance>
+<instance part="GND2" gate="1" x="139.7" y="2.54" smashed="yes">
+<attribute name="VALUE" x="143.34" y="0.5" size="1.778" layer="96" rot="R180"/>
+</instance>
+<instance part="GND3" gate="1" x="20.32" y="-33.02" smashed="yes" rot="R270">
+<attribute name="VALUE" x="18.28" y="-36.66" size="1.778" layer="96" rot="R90"/>
+</instance>
+<instance part="GND4" gate="1" x="27.94" y="20.32" smashed="yes">
+<attribute name="VALUE" x="31.58" y="18.28" size="1.778" layer="96" rot="R180"/>
+</instance>
+<instance part="GND7" gate="1" x="27.94" y="35.56" smashed="yes">
+<attribute name="VALUE" x="31.58" y="33.52" size="1.778" layer="96" rot="R180"/>
+</instance>
+<instance part="GND8" gate="1" x="27.94" y="53.34" smashed="yes">
+<attribute name="VALUE" x="31.58" y="51.3" size="1.778" layer="96" rot="R180"/>
+</instance>
 <instance part="OK1" gate="A" x="5.08" y="73.66" smashed="yes">
 <attribute name="NAME" x="-1.905" y="79.375" size="1.778" layer="95"/>
@@
 <attribute name="NAME" x="-1.905" y="31.115" size="1.778" layer="95"/>
 <attribute name="VALUE" x="-1.905" y="17.78" size="1.778" layer="96"/>
-</instance>
-<instance part="RTC" gate="G$1" x="99.06" y="0" smashed="yes">
-<attribute name="VALUE" x="97.79" y="-10.16" size="1.778" layer="96"/>
-<attribute name="NAME" x="97.79" y="8.382" size="1.778" layer="95"/>
-</instance>
-<instance part="COM_FUENTE" gate="1" x="-53.34" y="73.66" smashed="yes">
-<attribute name="VALUE" x="-54.61" y="63.5" size="1.778" layer="96"/>
-<attribute name="NAME" x="-54.61" y="79.502" size="1.778" layer="95"/>
-</instance>
-<instance part="+3V3" gate="G$1" x="129.54" y="-2.54" smashed="yes">
-<attribute name="VALUE" x="132.1" y="-0.04" size="1.778" layer="96" rot="R180"/>
-</instance>
-<instance part="GND2" gate="1" x="139.7" y="2.54" smashed="yes">
-<attribute name="VALUE" x="143.34" y="0.5" size="1.778" layer="96" rot="R180"/>
-</instance>
-<instance part="GND3" gate="1" x="20.32" y="-33.02" smashed="yes" rot="R270">
-<attribute name="VALUE" x="18.28" y="-36.66" size="1.778" layer="96" rot="R90"/>
-</instance>
-<instance part="GND4" gate="1" x="27.94" y="20.32" smashed="yes">
-<attribute name="VALUE" x="31.58" y="18.28" size="1.778" layer="96" rot="R180"/>
-</instance>
-<instance part="GND7" gate="1" x="27.94" y="35.56" smashed="yes">
-<attribute name="VALUE" x="31.58" y="33.52" size="1.778" layer="96" rot="R180"/>
-</instance>
-<instance part="GND8" gate="1" x="27.94" y="53.34" smashed="yes">
-<attribute name="VALUE" x="31.58" y="51.3" size="1.778" layer="96" rot="R180"/>
 </instance>
 </instances>
@@
 </segment>
 <segment>
-<pinref part="OK2" gate="B" pin="EMIT"/>
 <wire x1="12.7" y1="22.86" x2="27.94" y2="22.86" width="0.1524" layer="91"/>
 <pinref part="GND4" gate="1" pin="GNDA"/>
-</segment>
-<segment>
-<pinref part="OK2" gate="A" pin="EMIT"/>
+<pinref part="OK2" gate="B" pin="EMIT"/>
+</segment>
+<segment>
 <wire x1="12.7" y1="38.1" x2="27.94" y2="38.1" width="0.1524" layer="91"/>
 <pinref part="GND7" gate="1" pin="GNDA"/>
-</segment>
-<segment>
-<pinref part="OK1" gate="B" pin="EMIT"/>
+<pinref part="OK2" gate="A" pin="EMIT"/>
+</segment>
+<segment>
 <wire x1="12.7" y1="55.88" x2="27.94" y2="55.88" width="0.1524" layer="91"/>
 <pinref part="GND8" gate="1" pin="GNDA"/>
+<pinref part="OK1" gate="B" pin="EMIT"/>
 </segment>
 </net>
@@
 </segment>
 </net>
-<net name="N$1" class="0">
+<net name="N$1" class="2">
 <segment>
 <pinref part="COM_FUENTE" gate="1" pin="4"/>
 <wire x1="-45.72" y1="76.2" x2="-12.7" y2="76.2" width="0.1524" layer="91"/>
 <wire x1="-12.7" y1="76.2" x2="-12.7" y2="60.96" width="0.1524" layer="91"/>
+<wire x1="-12.7" y1="60.96" x2="-5.08" y2="60.96" width="0.1524" layer="91"/>
 <pinref part="OK1" gate="B" pin="A"/>
-<wire x1="-12.7" y1="60.96" x2="-5.08" y2="60.96" width="0.1524" layer="91"/>
-</segment>
-</net>
-<net name="N$2" class="0">
+</segment>
+</net>
+<net name="N$2" class="2">
 <segment>
 <pinref part="COM_FUENTE" gate="1" pin="3"/>
 <wire x1="-45.72" y1="73.66" x2="-15.24" y2="73.66" width="0.1524" layer="91"/>
-<pinref part="OK2" gate="A" pin="A"/>
 <wire x1="-15.24" y1="73.66" x2="-15.24" y2="43.18" width="0.1524" layer="91"/>
 <wire x1="-15.24" y1="43.18" x2="-5.08" y2="43.18" width="0.1524" layer="91"/>
-</segment>
-</net>
-<net name="N$3" class="0">
+<pinref part="OK2" gate="A" pin="A"/>
+</segment>
+</net>
+<net name="N$3" class="2">
 <segment>
 <pinref part="COM_FUENTE" gate="1" pin="2"/>
 <wire x1="-45.72" y1="71.12" x2="-20.32" y2="71.12" width="0.1524" layer="91"/>
 <wire x1="-20.32" y1="71.12" x2="-20.32" y2="27.94" width="0.1524" layer="91"/>
+<wire x1="-20.32" y1="27.94" x2="-5.08" y2="27.94" width="0.1524" layer="91"/>
 <pinref part="OK2" gate="B" pin="A"/>
-<wire x1="-20.32" y1="27.94" x2="-5.08" y2="27.94" width="0.1524" layer="91"/>
-</segment>
-</net>
-<net name="GND_FUENTE" class="0">
+</segment>
+</net>
+<net name="GND_FUENTE" class="2">
 <segment>
 <pinref part="COM_FUENTE" gate="1" pin="1"/>
 <wire x1="-45.72" y1="68.58" x2="-27.94" y2="68.58" width="0.1524" layer="91"/>
 <wire x1="-27.94" y1="68.58" x2="-27.94" y2="55.88" width="0.1524" layer="91"/>
-<pinref part="OK2" gate="B" pin="C"/>
 <wire x1="-27.94" y1="55.88" x2="-27.94" y2="38.1" width="0.1524" layer="91"/>
 <wire x1="-27.94" y1="38.1" x2="-27.94" y2="22.86" width="0.1524" layer="91"/>
 <wire x1="-27.94" y1="22.86" x2="-5.08" y2="22.86" width="0.1524" layer="91"/>
-<pinref part="OK1" gate="B" pin="C"/>
 <wire x1="-5.08" y1="55.88" x2="-27.94" y2="55.88" width="0.1524" layer="91"/>
 <junction x="-27.94" y="55.88"/>
-<pinref part="OK2" gate="A" pin="C"/>
 <wire x1="-5.08" y1="38.1" x2="-27.94" y2="38.1" width="0.1524" layer="91"/>
 <junction x="-27.94" y="38.1"/>
 <label x="-45.72" y="68.58" size="1.778" layer="95"/>
+<pinref part="OK1" gate="B" pin="C"/>
+<pinref part="OK2" gate="A" pin="C"/>
+<pinref part="OK2" gate="B" pin="C"/>
 </segment>
 </net>
 <net name="C_OPTO2" class="2">
 <segment>
-<pinref part="OK2" gate="A" pin="COL"/>
 <wire x1="12.7" y1="43.18" x2="27.94" y2="43.18" width="0.1524" layer="91"/>
 <label x="27.94" y="43.18" size="1.27" layer="95" xref="yes"/>
-</segment>
-<segment>
-<pinref part="SV2" gate="1" pin="14"/>
-<wire x1="38.1" y1="-60.96" x2="33.02" y2="-60.96" width="0.1524" layer="91"/>
-<label x="33.02" y="-60.96" size="1.27" layer="95" rot="R180" xref="yes"/>
+<pinref part="OK2" gate="A" pin="COL"/>
+<label x="27.94" y="43.18" size="1.27" layer="95" xref="yes"/>
+<label x="33.02" y="-66.04" size="1.27" layer="95" rot="R180" xref="yes"/>
+</segment>
+<segment>
+<pinref part="SV2" gate="1" pin="16"/>
+<wire x1="33.02" y1="-66.04" x2="38.1" y2="-66.04" width="0.1524" layer="91"/>
 </segment>
 </net>
 <net name="C_OPTO1" class="2">
 <segment>
-<pinref part="OK1" gate="B" pin="COL"/>
 <wire x1="12.7" y1="60.96" x2="27.94" y2="60.96" width="0.1524" layer="91"/>
 <label x="27.94" y="60.96" size="1.27" layer="95" xref="yes"/>
+<pinref part="OK1" gate="B" pin="COL"/>
 </segment>
 <segment>
@@
 <net name="C_OPTO3" class="2">
 <segment>
-<pinref part="OK2" gate="B" pin="COL"/>
 <wire x1="12.7" y1="27.94" x2="27.94" y2="27.94" width="0.1524" layer="91"/>
 <label x="27.94" y="27.94" size="1.27" layer="95" xref="yes"/>
-</segment>
-<segment>
-<pinref part="SV1" gate="1" pin="12"/>
-<wire x1="76.2" y1="-55.88" x2="73.66" y2="-55.88" width="0.1524" layer="91"/>
-<label x="73.66" y="-55.88" size="1.27" layer="95" rot="R180" xref="yes"/>
-</segment>
-</net>
+<pinref part="OK2" gate="B" pin="COL"/>
+<label x="33.02" y="-68.58" size="1.27" layer="95" rot="R180" xref="yes"/>
+</segment>
+<segment>
+<pinref part="SV2" gate="1" pin="17"/>
+<wire x1="33.02" y1="-68.58" x2="38.1" y2="-68.58" width="0.1524" layer="91"/>
+</segment>
+</net>
